Commit message: feat(hito1): agrega geometria visual basica al modelo URDF

File: 2-2026/IMT342/equipo/hitos/hito1/irb120_description/urdf/irb120.urdf (robot description, URDF)
Before this commit: robot irb120, 7 links, 6 joints
Links:
- link link_1: geometry visual cylinder length=0.290 radius=0.025
- link link_2: geometry visual cylinder length=0.270 radius=0.025
- link link_3: geometry visual cylinder length=0.070 radius=0.025
- link link_4: geometry visual cylinder length=0.302 radius=0.025
- link link_5: geometry visual cylinder length=0.072 radius=0.025

Commit message: feat(hito1): integra mallas visuales del IRB 120

File: 2-2026/IMT342/equipo/hitos/hito1/irb120_description/urdf/irb120.urdf (robot description, URDF)
Before this commit: robot irb120, 7 links, 6 joints
Links:
- link base_link: geometry visual mesh filename=package://irb120_description/meshes/visual/base_link.stl
- link link_1: geometry visual mesh filename=package://irb120_description/meshes/visual/link_1.stl
- link link_2: geometry visual mesh filename=package://irb120_description/meshes/visual/link_2.stl
- link link_3: geometry visual mesh filename=package://irb120_description/meshes/visual/link_3.stl
- link link_4: geometry visual mesh filename=package://irb120_description/meshes/visual/link_4.stl
- link link_5: geometry visual mesh filename=package://irb120_description/meshes/visual/link_5.stl
- link link_6: geometry visual mesh filename=package://irb120_description/meshes/visual/link_6.stl

Commit message: feat(hito1): integra mallas de colision del IRB 120

File: 2-2026/IMT342/equipo/hitos/hito1/irb120_description/urdf/irb120.urdf (robot description, URDF)
Before this commit: robot irb120, 7 links, 6 joints
Links:
- link base_link: geometry collision mesh filename=package://irb120_description/meshes/collision/base_link.stl; visual mesh filename=package://irb120_description/meshes/visual/base_link.stl
- link link_1: geometry collision mesh filename=package://irb120_description/meshes/collision/link_1.stl; visual mesh filename=package://irb120_description/meshes/visual/link_1.stl
- link link_2: geometry collision mesh filename=package://irb120_description/meshes/collision/link_2.stl; visual mesh filename=package://irb120_description/meshes/visual/link_2.stl
- link link_3: geometry collision mesh filename=package://irb120_description/meshes/collision/link_3.stl; visual mesh filename=package://irb120_description/meshes/visual/link_3.stl
- link link_4: geometry collision mesh filename=package://irb120_description/meshes/collision/link_4.stl; visual mesh filename=package://irb120_description/meshes/visual/link_4.stl
- link link_5: geometry collision mesh filename=package://irb120_description/meshes/collision/link_5.stl; visual mesh filename=package://irb120_description/meshes/visual/link_5.stl
- link link_6: geometry collision mesh filename=package://irb120_description/meshes/collision/link_6.stl; visual mesh filename=package://irb120_description/meshes/visual/link_6.stl

Commit message: feat(hito1): agrega frame terminal compatible con D-H

File: 2-2026/IMT342/equipo/hitos/hito1/irb120_description/urdf/irb120.urdf (robot description, URDF)
Before this commit: robot irb120, 7 links, 6 joints
Links:
- added link dh_frame_6
Joints:
- added joint link6_to_dh_frame_6: type fixed, parent link_6, child dh_frame_6, origin xyz=0 0 0 rpy=0 -1.5707963267948966 3.141592653589793

Commit message: feat(hito1): agrega pinza provisional y frame TCP

File: 2-2026/IMT342/equipo/hitos/hito1/irb120_description/urdf/irb120.urdf (robot description, URDF)
Before this commit: robot irb120, 8 links, 7 joints
Links:
- added link gripper_base; collision box size=0.060 0.050 0.060; visual box size=0.060 0.050 0.060
- added link tcp
Joints:
- added joint dh6_to_gripper: type fixed, parent dh_frame_6, child gripper_base, origin xyz=0 0 0 rpy=0 0 0
- added joint gripper_to_tcp: type fixed, parent gripper_base, child tcp, origin xyz=0 0 0.120 rpy=0 0 0
